File: hardware/epaper-breakout/_autosave-epaper-breakout.kicad_pcb (KiCad board)
At the start: 2 copper layers, 99.6 x 31.2 mm, 68 parts, among them J1 XF2M-3315-1A, J2 C10418, J3 Conn_02x06_Counter_Clockwise, J4 ED060SC4, Q1 IRLML6402, U1 MCP1700-3302E_SOT23, U2 LT1945, U3 LT1945, U5 ESP32-WROVER, U6 CH330N, U7 LM358, U8 74HC4094-normal, U9 MCP9700AT-ETT

Commit message: add preliminary 3rd hardware revision
*This is currently untested!*
A new revision of the hardware, reducing power consumption.
Parts:
- R18: value 300k -> 110k
- R19: value 28k -> 10k
Changed lines of the file:
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@@
       (effects (font (size 1 1) (thickness 0.15)))
     )
-    (fp_text value 28k (at 0 1.65 90) (layer F.Fab)
+    (fp_text value 10k (at 0 1.65 90) (layer F.Fab)
       (effects (font (size 1 1) (thickness 0.15)))
     )
@@
       (effects (font (size 1 1) (thickness 0.15)))
     )
-    (fp_text value 300k (at 0 1.65 90) (layer F.Fab)
+    (fp_text value 110k (at 0 1.65 90) (layer F.Fab)
       (effects (font (size 1 1) (thickness 0.15)))
     )
