File: hardware/epaper-breakout/epaper-breakout.sch (KiCad schematic (older format))
At the start: 60 parts, among them J1 XF2M-3315-1A, J2 C10418, J3 Conn_02x05_Counter_Clockwise, J4 ED060SC4, Q1 IRLML6402, U1 LT1086-3.3, U2 LT1945, U3 L7915, U4 L7815, U5 ESP32-WROVER, U6 CH330N, U7 LM358, U8 74HC4094-normal, U9 MCP9700AT-ETT

Commit message: add preliminary 3rd hardware revision
*This is currently untested!*
A new revision of the hardware, reducing power consumption.
Parts:
- removed C6: 0.33uF, Capacitor_SMD:C_0603_1608Metric, symbol Device:C
- removed J3: Conn_02x05_Counter_Clockwise, Connector_PinHeader_2.54mm:PinHeader_2x05_P2.54mm_Vertical, symbol Connector_Generic:Conn_02x05_Counter_Clockwise
- removed JP1: 5v or 3v to LT1945, Jumper:SolderJumper-3_P1.3mm_Bridged12_RoundedPad1.0x1.5mm, symbol Jumper:SolderJumper_3_Bridged12
- removed R1: 10k, Resistor_SMD:R_0805_2012Metric, symbol Device:R
- removed U1: LT1086-3.3, Package_TO_SOT_SMD:TO-252-2, symbol Regulator_Linear:LT1086-3.3
- removed U3: L7915, Package_TO_SOT_SMD:TO-252-2, symbol Regulator_Linear:L7915
- removed U4: L7815, Package_TO_SOT_SMD:TO-252-2, symbol Regulator_Linear:L7815
- added C19, C20: 1uF, Capacitor_SMD:C_0603_1608Metric, symbol Device:C
- added C6: 4.7uF, Capacitor_SMD:C_0603_1608Metric, symbol Device:CP
- added D4, D5, D6: MBR0540, Diode_SMD:D_SOD-123, symbol Diode:MBR0540
- added J3: Conn_02x06_Counter_Clockwise, Connector_PinHeader_2.54mm:PinHeader_2x06_P2.54mm_Vertical, symbol Connector_Generic:Conn_02x06_Counter_Clockwise
- added L3, L4: 22uH, Inductor_SMD:L_6.3x6.3_H3, symbol Device:L
- added R16: 300k, Resistor_SMD:R_0805_2012Metric, symbol Device:R
- added R17: 27k, Resistor_SMD:R_0805_2012Metric, symbol Device:R
- added R18: 110k, Resistor_SMD:R_0805_2012Metric, symbol Device:R
- added R19: 10k, Resistor_SMD:R_0805_2012Metric, symbol Device:R
- added U1: MCP1700-3302E_SOT23, Package_TO_SOT_SMD:SOT-23, symbol Regulator_Linear:MCP1700-3302E_SOT23
- added U3: LT1945, Package_SO:MSOP-10_3x3mm_P0.5mm, symbol Regulator_Switching:LT1945
- C10: value 1uF -> 4.7pF
- C11: value 1uF -> 100pF
- C7: value 0.33uF -> 0.1uF
- R8, R9: value 39k -> 10k
Connections:
- net labels added: A1, CTRL+15V, CTRL+22V, CTRL-15V, CTRL-20V, EPD_POWER
- net labels removed: CS0, EP_UD, NEG_CTRL, POS_CTRL
- wire segments 309 -> 357
Other:
- note removed: "Power +/-15V"
